Commit message: updated the filename

File: urdf/robo_serve.urdf (robot description, URDF)
Before this commit: robot modified_robo9_with_planning, 9 links, 8 joints
Links:
- link base_link: geometry collision mesh filename=package://robo_serve/meshes/base_link.STL; visual mesh filename=package://robo_serve/meshes/base_link.STL
- link base_to_first_link: geometry collision mesh filename=package://robo_serve/meshes/base_to_first_link.STL; visual mesh filename=package://robo_serve/meshes/base_to_first_link.STL
- link end_effector_link: geometry collision mesh filename=package://robo_serve/meshes/end_effector_link.STL; visual mesh filename=package://robo_serve/meshes/end_effector_link.STL
- link first_link: geometry collision mesh filename=package://robo_serve/meshes/first_link.STL; visual mesh filename=package://robo_serve/meshes/first_link.STL
- link left_wheel: geometry collision mesh filename=package://robo_serve/meshes/left_wheel.STL; visual mesh filename=package://robo_serve/meshes/left_wheel.STL
- link right_wheel: geometry collision mesh filename=package://robo_serve/meshes/right_wheel.STL; visual mesh filename=package://robo_serve/meshes/right_wheel.STL
- link second_link: geometry collision mesh filename=package://robo_serve/meshes/second_link.STL; visual mesh filename=package://robo_serve/meshes/second_link.STL
- link tray_diffusor: geometry collision mesh filename=package://robo_serve/meshes/tray_diffusor.STL; visual mesh filename=package://robo_serve/meshes/tray_diffusor.STL

File: urdf/robo_serve.xacro (robot description, xacro)
@@ -1,9 +1,9 @@
 <?xml version="1.0"?>
 <!-- Name your robot here -->
-<robot name ="modified_robo9_with_planning" xmlns:xacro="http://wiki.ros.org/xacro">
+<robot name ="robo_serve" xmlns:xacro="http://wiki.ros.org/xacro">
 <!-- Include your urdf files here -->
 	<!-- Include Robot's urdf filepath -->
 	<!-- Include Lidar's urdf filepath -->
-	<xacro:include filename="$(find modified_robo9_with_planning)/urdf/modified_robo9_with_planning.urdf"/>
+	<xacro:include filename="$(find robo_serve)/urdf/robo_serve.urdf"/>
 	<xacro:macro name="box_inertia" params="mass x y z">
         <inertia ixx="${mass*(y*y+z*z)/12}" ixy = "0" ixz = "0" iyy="${mass*(x*x+z*z)/12}" iyz = "0" izz="${mass*(x*x+y*y)/12}" />
@@ -32,5 +32,5 @@
 		<!-- <topic>__default_topic__</topic>/ -->
 		<plugin filename="libgazebo_ros_imu_sensor.so" name="imu_plugin">
-			<topicName>/modified_robo9_with_planning/imu</topicName>
+			<topicName>/robo_serve/imu</topicName>
 			<bodyName>imu_link</bodyName>
 			<updateRateHZ>10.0</updateRateHZ>
@@ -47,5 +47,5 @@
 	<gazebo>
 		<plugin name="gazebo_ros_control" filename="libgazebo_ros_control.so">
-			<robotNamespace>/modified_robo9_with_planning</robotNamespace>
+			<robotNamespace>/robo_serve</robotNamespace>
 			<robotSimType>gazebo_ros_control/DefaultRobotHWSim</robotSimType>
 			<legacyModeNS>true</legacyModeNS>
@@ -74,6 +74,6 @@
 			<wheelTorque>40</wheelTorque>
 			<wheelAcceleration>5.0</wheelAcceleration>
-			<commandTopic>/modified_robo9_with_planning/cmd_vel</commandTopic>
-			<odometryTopic>/modified_robo9_with_planning/odom</odometryTopic>
+			<commandTopic>/robo_serve/cmd_vel</commandTopic>
+			<odometryTopic>/robo_serve/odom</odometryTopic>
 			<odometryFrame>odom</odometryFrame>
 			<robotBaseFrame>dummy_link</robotBaseFrame>
